File: blink/blink - Copy.brd (EAGLE design)
At the start: 43.2 x 48.3 mm, 13 parts, among them T1 2N3904, T2 2N3904

Commit message: modified blink board
Routing:
- net +3V3: track 67.1 -> 91.7 mm
- net N$4: track 50.5 -> 30.0 mm
- net GND: track 66.4 -> 58.5 mm
- net N$5: track 29.8 -> 35.8 mm
- net N$1: track 22.6 -> 21.9 mm
